Commit message: modified urdf

File: data/urdf/red_robot.urdf (robot description, URDF)
Before this commit: robot red_robot, 36 links, 35 joints
Links:
- link AnkleCenter_L_Link: geometry collision mesh filename=package://hpp-timeopt-corba/meshes/AnkleCenter_L_Link.stl; visual mesh filename=package://hpp-timeopt-corba/meshes/AnkleCenter_L_Link.stl
- link AnkleCenter_R_Link: geometry visual mesh filename=package://hpp-timeopt-corba/meshes/AnkleCenter_R_Link.stl
- link AnkleRoll_L_Link: geometry collision mesh filename=package://hpp-timeopt-corba/meshes/AnkleRoll_L_Link.stl; visual mesh filename=package://hpp-timeopt-corba/meshes/AnkleRoll_L_Link.stl
- link AnkleRoll_R_Link: geometry collision mesh filename=package://hpp-timeopt-corba/meshes/AnkleRoll_R_Link.stl scale=1 1 1; visual mesh filename=package://hpp-timeopt-corba/meshes/AnkleRoll_R_Link.stl
- link Head: geometry collision mesh filename=package://hpp-timeopt-corba/meshes/head.stl; visual mesh filename=package://hpp-timeopt-corba/meshes/head.stl
- link HipCenter_L_Link: geometry visual mesh filename=package://hpp-timeopt-corba/meshes/HipCenter_L_Link.stl
- link HipCenter_R_Link: geometry visual mesh filename=package://hpp-timeopt-corba/meshes/HipCenter_R_Link.stl
- link HipRoll_L_Link: geometry visual mesh filename=package://hpp-timeopt-corba/meshes/HipRoll_L_Link.stl
- link HipRoll_R_link: geometry visual mesh filename=package://hpp-timeopt-corba/meshes/HipRoll_R_link.stl
- link Knee_L_Link: geometry collision mesh filename=package://hpp-timeopt-corba/meshes/Knee_L_Link.stl; visual mesh filename=package://hpp-timeopt-corba/meshes/Knee_L_Link.stl
- link Knee_R_Link: geometry visual mesh filename=package://hpp-timeopt-corba/meshes/Knee_R_Link.stl
- link L_armlink: geometry collision mesh filename=package://hpp-timeopt-corba/meshes/L_arm.stl; visual mesh filename=package://hpp-timeopt-corba/meshes/L_arm.stl
- link L_elbow: geometry collision mesh filename=package://hpp-timeopt-corba/meshes/L_elbow.stl; visual mesh filename=package://hpp-timeopt-corba/meshes/L_elbow.stl
- link L_forearm: geometry collision mesh filename=package://hpp-timeopt-corba/meshes/L_forearm.stl; visual mesh filename=package://hpp-timeopt-corba/meshes/L_forearm.stl
- link L_shoulder1: geometry collision mesh filename=package://hpp-timeopt-corba/meshes/L_shoulder1.stl; visual mesh filename=package://hpp-timeopt-corba/meshes/L_shoulder1.stl
- link L_shoulder2: geometry collision mesh filename=package://hpp-timeopt-corba/meshes/L_shoulder2.stl; visual mesh filename=package://hpp-timeopt-corba/meshes/L_shoulder2.stl
- link L_shoulder3: geometry collision mesh filename=package://hpp-timeopt-corba/meshes/L_shoulder3.stl; visual mesh filename=package://hpp-timeopt-corba/meshes/L_shoulder3.stl
- link L_wrist1: geometry collision mesh filename=package://hpp-timeopt-corba/meshes/L_wrist1.stl; visual mesh filename=package://hpp-timeopt-corba/meshes/L_wrist1.stl
- link L_wrist2: geometry collision mesh filename=package://hpp-timeopt-corba/meshes/L_wrist2.stl; visual mesh filename=package://hpp-timeopt-corba/meshes/L_wrist2.stl
- link Neck: geometry collision mesh filename=package://hpp-timeopt-corba/meshes/neck.stl; visual mesh filename=package://hpp-timeopt-corba/meshes/neck.stl
- link Pelvis_link: geometry collision mesh filename=package://hpp-timeopt-corba/meshes/Pelvis_link.stl; visual mesh filename=package://hpp-timeopt-corba/meshes/Pelvis_link.stl
- link R_armlink: geometry collision mesh filename=package://hpp-timeopt-corba/meshes/R_arm.stl; visual mesh filename=package://hpp-timeopt-corba/meshes/R_arm.stl
- link R_elbow: geometry collision mesh filename=package://hpp-timeopt-corba/meshes/R_elbow.stl; visual mesh filename=package://hpp-timeopt-corba/meshes/R_elbow.stl
- link R_forearm: geometry collision mesh filename=package://hpp-timeopt-corba/meshes/R_forearm.stl; visual mesh filename=package://hpp-timeopt-corba/meshes/R_forearm.stl
- link R_shoulder1: geometry collision mesh filename=package://hpp-timeopt-corba/meshes/R_shoulder1.stl; visual mesh filename=package://hpp-timeopt-corba/meshes/R_shoulder1.stl
- link R_shoulder2: geometry collision mesh filename=package://hpp-timeopt-corba/meshes/R_shoulder2.stl; visual mesh filename=package://hpp-timeopt-corba/meshes/R_shoulder2.stl
- link R_shoulder3: geometry collision mesh filename=package://hpp-timeopt-corba/meshes/R_shoulder3.stl; visual mesh filename=package://hpp-timeopt-corba/meshes/R_shoulder3.stl
- link R_wrist1: geometry collision mesh filename=package://hpp-timeopt-corba/meshes/R_wrist1.stl; visual mesh filename=package://hpp-timeopt-corba/meshes/R_wrist1.stl
- link R_wrist2: geometry collision mesh filename=package://hpp-timeopt-corba/meshes/R_wrist2.stl; visual mesh filename=package://hpp-timeopt-corba/meshes/R_wrist2.stl
- link Thigh_L_Link: geometry visual mesh filename=package://hpp-timeopt-corba/meshes/Thigh_L_Link.stl
- link Thigh_R_Link: geometry visual mesh filename=package://hpp-timeopt-corba/meshes/Thigh_R_Link.stl
- link Upperbody: geometry collision mesh filename=package://hpp-timeopt-corba/meshes/upperbody.stl; visual mesh filename=package://hpp-timeopt-corba/meshes/upperbody.stl
- link Waist1: geometry collision mesh filename=package://hpp-timeopt-corba/meshes/waist1.stl; visual mesh filename=package://hpp-timeopt-corba/meshes/waist1.stl
- link Waist2: geometry collision mesh filename=package://hpp-timeopt-corba/meshes/waist2.stl; visual mesh filename=package://hpp-timeopt-corba/meshes/waist2.stl
