Commit message: modified server for using rbprm-server

File: data/urdf/red_lleg.urdf (robot description, URDF)
Before this commit: robot chair, 1 links, 0 joints
Links:
- link base_link: geometry collision mesh filename=package://hpp-timeopt-corba/meshes/red/red_lleg.stl; visual mesh filename=package://hpp-timeopt-corba/meshes/red/red_lleg.stl

File: data/urdf/red_rleg.urdf (robot description, URDF)
Before this commit: robot chair, 1 links, 0 joints
Links:
- link base_link: geometry collision mesh filename=package://hpp-timeopt-corba/meshes/red/red_rleg.stl; visual mesh filename=package://hpp-timeopt-corba/meshes/red/red_rleg.stl

File: data/urdf/red_trunk.urdf (robot description, URDF)
Before this commit: robot chair, 1 links, 0 joints
Links:
- link base_link: geometry collision mesh filename=package://hpp-timeopt-corba/meshes/red/trunk.stl; visual mesh filename=package://hpp-timeopt-corba/meshes/red/red_whole.stl
